File: KiCad/Onboard_Vehicle_PCB/Onboard_Vehicle_PCB.kicad_pcb (KiCad board)
At the start: 2 copper layers, 100 x 70 mm, 8 parts, among them J1 Teensy-Left, J2 Teensy-Right, J3 S3:0 (L), J4 S3:0 (M), J5 S3:0 (R), J6 S3:0 (A), J7 OUT-ARML, J8 5V-Conn

Commit message: PCB v1 WIP
Parts:
- added J9: GND-Conn, Connector_PinHeader_2.54mm:PinHeader_1x06_P2.54mm_Vertical, F.Cu at (108.0, 89.8)
- added R1: 330, Resistor_THT:R_Axial_DIN0204_L3.6mm_D1.6mm_P7.62mm_Horizontal, F.Cu at (87.9, 91.8)
- added R2: 330, Resistor_THT:R_Axial_DIN0204_L3.6mm_D1.6mm_P7.62mm_Horizontal, F.Cu at (87.9, 95.0)
- added SW1: Start_Button, Button_Switch_THT:SW_PUSH_6mm, F.Cu at (77.9, 92.3)
- added SW2: Calibration_Button, Button_Switch_THT:SW_PUSH_6mm, F.Cu at (77.9, 100.8)
Connections:
- net /14 renamed /DATA_1
- net /15 renamed /DATA_2
- net /16 renamed /ENA
- net /17 renamed /ENB
- net /18 renamed /IN1
- net /19 renamed /IN2
- net /20 renamed /IN3
- net /21 renamed /IN4
- net /37 renamed /Trig
- net /38 renamed /Echo
- J1 pad 16: unconnected-(J1-Pin_16-Pad16) -> /PRES
- J1 pad 19: /27 -> /CAL_BUTTON
- J1 pad 20: /28 -> /START_BUTTON
- J1 pad 21: /29 -> /Aout
- J1 pad 22: /30 -> /Rout
- J1 pad 23: /31 -> /Mout
- J1 pad 24: /32 -> /Lout
- J1 pad 5: unconnected-(J1-Pin_5-Pad5) -> /3
- J2 pad 1: /33 -> /S0
- J2 pad 2: /34 -> /S1
- J2 pad 3: /35 -> /S2
- J2 pad 4: /36 -> /S3

Commit message: Commit 4/25
Parts:
- J8: value 5V-Conn -> 5V
- J9: value GND-Conn -> GND
- R1, R2: footprint Resistor_THT:R_Axial_DIN0204_L3.6mm_D1.6mm_P7.62mm_Horizontal -> Resistor_THT:R_Axial_DIN0207_L6.3mm_D2.5mm_P10.16mm_Horizontal
- moved J1 68.4 mm to (119.6, 53.5), turned to -90 degrees
- moved J2 67.9 mm to (119.6, 71.3), turned to -90 degrees
- moved J8 59.0 mm to (58.5, 95.1), turned to 180 degrees
- moved J9 54.3 mm to (54.0, 95.0), turned to 180 degrees
- moved J7 30.1 mm to (128.0, 62.0)
- moved R1 20.2 mm to (75.5, 75.9), turned to -90 degrees
- moved SW1 17.7 mm to (64.0, 81.2)
- moved SW2 17.3 mm to (64.0, 90.5)
- moved J6 14.8 mm to (121.5, 85.6), turned to 180 degrees
- moved R2 13.8 mm to (75.5, 88.9), turned to -90 degrees
- moved J3 12.2 mm to (133.5, 85.6), turned to 180 degrees
- moved J5 6.85 mm to (125.5, 85.6), turned to 180 degrees
- moved J4 4.81 mm to (129.5, 85.6), turned to 180 degrees
Connections:
- J1 pad 19: /CAL_BUTTON -> /27
- J1 pad 20: /START_BUTTON -> /28
- J2 pad 20: /22 -> /START_BUTTON
- J2 pad 21: /23 -> /CAL_BUTTON
Other:
- board size 100 x 70 mm -> 100 x 80 mm
