File: KiCad/Onboard_Vehicle_PCB/Onboard_Vehicle_PCB.kicad_sch (KiCad schematic)
At the start: 8 parts, among them J1 Teensy-Left, J2 Teensy-Right, J3 S3:0 (L), J4 S3:0 (M), J5 S3:0 (R), J6 S3:0 (A), J7 OUT-ARML, J8 5V-Conn

Commit message: PCB v1 WIP
Parts:
- added J9: GND-Conn, Connector_PinHeader_2.54mm:PinHeader_1x06_P2.54mm_Vertical, symbol Connector_Generic:Conn_01x06
- added R1, R2: 330, Resistor_THT:R_Axial_DIN0204_L3.6mm_D1.6mm_P7.62mm_Horizontal, symbol Device:R
- added SW1: Start_Button, Button_Switch_THT:SW_PUSH_6mm, symbol Switch:SW_Push
- added SW2: Calibration_Button, Button_Switch_THT:SW_PUSH_6mm, symbol Switch:SW_Push
Connections:
- net 29 is gone; now on net Aout: J1.21 (Pin_21)
- net 30 is gone; now on net Rout: J1.22 (Pin_22)
- net 31 is gone; now on net Mout: J1.23 (Pin_23)
- net 32 is gone; now on net Lout: J1.24 (Pin_24)
- net +5V: now also SW1.1, SW2.1
- net 3: now also J1.5 (Pin_5)
- net GND: now also J9.1 (Pin_1), J9.2 (Pin_2), J9.3 (Pin_3), J9.4 (Pin_4), J9.5 (Pin_5), J9.6 (Pin_6), R1.1, R2.1
- net PRES: now reaches J1.16 (Pin_16)
- net 27 renamed CAL_BUTTON
- net CAL_BUTTON: now also R2.2, SW2.2
- net 28 renamed START_BUTTON
- net START_BUTTON: now also R1.2, SW1.2
- net 38 renamed Echo
Other:
- note added: "(24)"
- note added: "(27)"
- note added: "(28)"
- note added: "(29)"
- note added: "(30)"
- note added: "(31)"
- note added: "(32)"
- note added: "(38)"
- note added: "Buttons"
- note added: "Color Sensor Array"
- moved on the sheet: J3, J4, J5, J6, J7, J8

Commit message: Commit 4/25
Parts:
- R1, R2: footprint Resistor_THT:R_Axial_DIN0204_L3.6mm_D1.6mm_P7.62mm_Horizontal -> Resistor_THT:R_Axial_DIN0207_L6.3mm_D2.5mm_P10.16mm_Horizontal
Connections:
- net 22 is gone; now on net START_BUTTON: J2.20 (Pin_20)
- net 23 is gone; now on net CAL_BUTTON: J2.21 (Pin_21)
- net CAL_BUTTON: no longer J1.19 (Pin_19)
- net START_BUTTON: no longer J1.20 (Pin_20)
- net 4 renamed IN4_R
- net 5 renamed IN3_R
- net 6 renamed IN2_R
- net 7 renamed IN1_R
- net 8 renamed ENB_R
- net 9 renamed ENA_R
- net DATA_1 renamed DATA_ARM
- net DATA_2 renamed DATA_GRIP
- net ENA renamed ENA_L
- net ENB renamed ENB_L
- net IN1 renamed IN1_L
- net IN2 renamed IN2_L
- net IN3 renamed IN3_L
- net IN4 renamed IN4_L
- new net 27: J1.19 (Pin_19)
- new net 28: J1.20 (Pin_20)
Other:
- note added: "(22)"
- note added: "(23)"
- note added: "(4)"
- note added: "(5)"
- note added: "(6)"
- note added: "(7)"
- note added: "(8)"
- note added: "(9)"
- note removed: "(27)"
- note removed: "(28)"
Changed lines of the file:
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@@
 	(text "(19)"
 		(exclude_from_sim no)
-		(at 87.122 55.118 0)
-		(effects
-			(font
-				(size 1.27 1.27)
-			)
-		)
-	)
-	(text "(27)"
-		(exclude_from_sim no)
-		(at 29.718 83.058 0)
+		(at 95.25 55.118 0)
+		(effects
+			(font
+				(size 1.27 1.27)
+			)
+		)
+	)
+	(text "(23)"
+		(exclude_from_sim no)
+		(at 95.25 44.704 0)
 		(effects
 			(font
@@
 	(text "(17)\n"
 		(exclude_from_sim no)
-		(at 87.122 60.198 0)
+		(at 95.25 60.198 0)
 		(effects
 			(font
@@
 		)
 	)
+	(text "(5)\n"
+		(exclude_from_sim no)
+		(at 36.576 52.324 0)
+		(effects
+			(font
+				(size 1.27 1.27)
+			)
+		)
+	)
+	(text "(9)"
+		(exclude_from_sim no)
+		(at 36.83 62.738 0)
+		(effects
+			(font
+				(size 1.27 1.27)
+			)
+		)
+	)
+	(text "(7)"
+		(exclude_from_sim no)
+		(at 36.83 57.404 0)
+		(effects
+			(font
+				(size 1.27 1.27)
+			)
+		)
+	)
 	(text "(30)"
 		(exclude_from_sim no)
@@
 	(text "(15)\n"
 		(exclude_from_sim no)
-		(at 87.122 65.278 0)
+		(at 95.25 65.278 0)
 		(effects
 			(font
@@
 	(text "(18)"
 		(exclude_from_sim no)
-		(at 87.122 57.658 0)
+		(at 95.25 57.658 0)
 		(effects
 			(font
@@
 		)
 	)
+	(text "(6)\n"
+		(exclude_from_sim no)
+		(at 36.83 55.118 0)
+		(effects
+			(font
+				(size 1.27 1.27)
+			)
+		)
+	)
 	(text "Color Sensor Array"
 		(exclude_from_sim no)
@@
 		)
 	)
-	(text "(28)"
-		(exclude_from_sim no)
-		(at 29.718 85.598 0)
+	(text "(22)"
+		(exclude_from_sim no)
+		(at 95.25 47.244 0)
 		(effects
 			(font
@@
 	(text "(16)\n"
 		(exclude_from_sim no)
-		(at 87.122 62.738 0)
+		(at 95.25 62.738 0)
 		(effects
 			(font
@@
 	(text "(21)"
 		(exclude_from_sim no)
-		(at 87.122 50.038 0)
+		(at 95.25 50.038 0)
+		(effects
+			(font
+				(size 1.27 1.27)
+			)
+		)
+	)
+	(text "(4)"
+		(exclude_from_sim no)
+		(at 36.576 49.784 0)
 		(effects
 			(font
@@
 	(text "(20)"
 		(exclude_from_sim no)
-		(at 87.122 52.578 0)
+		(at 95.25 52.578 0)
 		(effects
 			(font
@@
 		)
 	)
+	(text "(8)"
+		(exclude_from_sim no)
+		(at 36.83 60.198 0)
+		(effects
+			(font
+				(size 1.27 1.27)
+			)
+		)
+	)
 	(text "(31)"
 		(exclude_from_sim no)
@@
 	(text "(14)\n"
 		(exclude_from_sim no)
-		(at 87.122 67.818 0)
+		(at 95.25 67.818 0)
 		(effects
 			(font
@@
 		)
 	)
+	(label "IN3_R"
+		(at 45.72 53.34 180)
+		(effects
+			(font
+				(size 1.27 1.27)
+			)
+			(justify right bottom)
+		)
+	)
 	(label "12"
 		(at 45.72 71.12 180)
@@
 		)
 	)
-	(label "ENA"
+	(label "ENA_L"
 		(at 77.47 63.5 0)
 		(effects
@@
 		)
 	)
-	(label "22"
-		(at 77.47 48.26 0)
+	(label "28"
+		(at 45.72 86.36 180)
+		(effects
+			(font
+				(size 1.27 1.27)
+			)
+			(justify right bottom)
+		)
+	)
+	(label "CAL_BUTTON"
+		(at 77.47 45.72 0)
 		(effects
 			(font
@@
 		)
 	)
-	(label "DATA_1"
+	(label "DATA_ARM"
 		(at 77.47 68.58 0)
 		(effects
@@
 		)
 	)
-	(label "7"
-		(at 45.72 58.42 180)
-		(effects
-			(font
-				(size 1.27 1.27)
-			)
-			(justify right bottom)
-		)
-	)
 	(label "39"
 		(at 77.47 81.28 0)
@@
 		)
 	)
-	(label "6"
-		(at 45.72 55.88 180)
-		(effects
-			(font
-				(size 1.27 1.27)
-			)
-			(justify right bottom)
-		)
-	)
 	(label "S0"
 		(at 212.09 99.06 180)
@@
 		)
 	)
-	(label "IN2"
+	(label "IN2_L"
 		(at 77.47 55.88 0)
 		(effects
@@
 		)
 	)
-	(label "8"
+	(label "ENB_R"
 		(at 45.72 60.96 180)
 		(effects
@@
 		)
 	)
-	(label "IN4"
+	(label "IN4_L"
 		(at 77.47 50.8 0)
 		(effects
@@
 		)
 	)
-	(label "CAL_BUTTON"
-		(at 45.72 83.82 180)
+	(label "ENA_R"
+		(at 45.72 63.5 180)
 		(effects
 			(font
@@
 		)
 	)
-	(label "IN1"
+	(label "IN1_L"
 		(at 77.47 58.42 0)
 		(effects
@@
 			)
 			(justify left bottom)
-		)
-	)
-	(label "5"
-		(at 45.72 53.34 180)
-		(effects
-			(font
-				(size 1.27 1.27)
-			)
-			(justify right bottom)
 		)
 	)
@@
 	)
 	(label "START_BUTTON"
-		(at 45.72 86.36 180)
-		(effects
-			(font
-				(size 1.27 1.27)
-			)
-			(justify right bottom)
+		(at 77.47 48.26 0)
+		(effects
+			(font
+				(size 1.27 1.27)
+			)
+			(justify left bottom)
 		)
 	)
@@
 		)
 	)
-	(label "ENB"
+	(label "IN1_R"
+		(at 45.72 58.42 180)
+		(effects
+			(font
+				(size 1.27 1.27)
+			)
+			(justify right bottom)
+		)
+	)
+	(label "ENB_L"
 		(at 77.47 60.96 0)
 		(effects
@@
 			)
 			(justify left bottom)
+		)
+	)
+	(label "IN2_R"
+		(at 45.72 55.88 180)
+		(effects
+			(font
+				(size 1.27 1.27)
+			)
+			(justify right bottom)
 		)
 	)
@@
 		)
 	)
-	(label "23"
-		(at 77.47 45.72 0)
-		(effects
-			(font
-				(size 1.27 1.27)
-			)
-			(justify left bottom)
+	(label "27"
+		(at 45.72 83.82 180)
+		(effects
+			(font
+				(size 1.27 1.27)
+			)
+			(justify right bottom)
+		)
+	)
+	(label "IN4_R"
+		(at 45.72 50.8 180)
+		(effects
+			(font
+				(size 1.27 1.27)
+			)
+			(justify right bottom)
 		)
 	)
@@
 		)
 	)
-	(label "4"
-		(at 45.72 50.8 180)
-		(effects
-			(font
-				(size 1.27 1.27)
-			)
-			(justify right bottom)
-		)
-	)
 	(label "S3"
 		(at 208.28 91.44 180)
@@
 		)
 	)
-	(label "9"
-		(at 45.72 63.5 180)
-		(effects
-			(font
-				(size 1.27 1.27)
-			)
-			(justify right bottom)
-		)
-	)
 	(label "Mout"
 		(at 45.72 93.98 180)
@@
 		)
 	)
-	(label "IN3"
+	(label "IN3_L"
 		(at 77.47 53.34 0)
 		(effects
@@
 		)
 	)
-	(label "DATA_2"
+	(label "DATA_GRIP"
 		(at 77.47 66.04 0)
 		(effects
@@
 			)
 		)
-		(property "Footprint" "Resistor_THT:R_Axial_DIN0204_L3.6mm_D1.6mm_P7.62mm_Horizontal"
+		(property "Footprint" "Resistor_THT:R_Axial_DIN0207_L6.3mm_D2.5mm_P10.16mm_Horizontal"
 			(at 84.328 139.7 90)
 			(effects
@@
 			)
 		)
-		(property "Footprint" "Resistor_THT:R_Axial_DIN0204_L3.6mm_D1.6mm_P7.62mm_Horizontal"
+		(property "Footprint" "Resistor_THT:R_Axial_DIN0207_L6.3mm_D2.5mm_P10.16mm_Horizontal"
 			(at 122.428 139.7 90)
 			(effects
